Commit message: feat(sim): drive base with wheel physics and diff_drive_controller
Replace the kinematic BaseVelocityPlugin freejoint override with real
velocity-actuated wheels: continuous wheel joints in the URDF, hinge +
friction-contact wheels and velocity actuators in the MJCF, and the
stock diff_drive_controller for cmd_vel and encoder odometry. Its odom
TF makes the odom_to_tf.py bridge and mujoco_plugins.yaml redundant.

Co-Authored-By: Claude Fable 5 <noreply@anthropic.com>
Claude-Session: https://claude.ai/code/session_01CWncjddFbcDzFPsMRYrkuq

File: mobile_manipulator_simulation/description/rox_diff_ur5e_control.urdf.xacro (robot description, xacro)
@@ -49,4 +49,16 @@
       <state_interface name="velocity"/>
     </joint>
+    <!-- Drive wheels: MJCF has 1:1 named <velocity> actuators; the velocity command
+         maps directly to ctrl. -->
+    <joint name="wheel_left_joint">
+      <command_interface name="velocity"/>
+      <state_interface name="position"/>
+      <state_interface name="velocity"/>
+    </joint>
+    <joint name="wheel_right_joint">
+      <command_interface name="velocity"/>
+      <state_interface name="position"/>
+      <state_interface name="velocity"/>
+    </joint>
     <!-- Mimic slaves: state-only so joint_state_broadcaster feeds robot_state_publisher.
          MuJoCo equality constraints drive them; MujocoSystemInterface registers them as

File: mobile_manipulator_simulation/description/rox_diff_ur5e_mujoco.urdf (robot description, URDF)
Before this commit: robot rox, 35 links, 34 joints
Links:
- link base_footprint: geometry collision mesh filename=package://mobile_manipulator_simulation/description/meshes/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 scale=0.1 0.1 0.1; visual mesh filename=package://mobile_manipulator_simulation/description/meshes/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 scale=0.1 0.1 0.1
- link cabinet_link: geometry collision mesh filename=package://mobile_manipulator_simulation/description/meshes/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 scale=0.1 0.1 0.1; visual mesh filename=package://mobile_manipulator_simulation/description/meshes/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 scale=0.1 0.1 0.1
- link caster_wheel_back_left_link: geometry collision sphere radius=0.124; visual mesh filename=package://mobile_manipulator_simulation/description/meshes/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 scale=0.001 0.001 0.001
- link caster_wheel_back_right_link: geometry collision sphere radius=0.124; visual mesh filename=package://mobile_manipulator_simulation/description/meshes/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 scale=0.001 0.001 0.001
- link caster_wheel_front_left_link: geometry collision sphere radius=0.124; visual mesh filename=package://mobile_manipulator_simulation/description/meshes/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 scale=0.001 0.001 0.001
- link caster_wheel_front_right_link: geometry collision sphere radius=0.124; visual mesh filename=package://mobile_manipulator_simulation/description/meshes/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 scale=0.001 0.001 0.001
- link lidar_1_link: geometry collision mesh filename=package://mobile_manipulator_simulation/description/meshes/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 scale=0.1 0.1 0.1; visual mesh filename=package://mobile_manipulator_simulation/description/meshes/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 scale=0.1 0.1 0.1
- link lidar_2_link: geometry collision mesh filename=package://mobile_manipulator_simulation/description/meshes/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 scale=0.1 0.1 0.1; visual mesh filename=package://mobile_manipulator_simulation/description/meshes/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 scale=0.1 0.1 0.1
- link robotiq_85_base_link: geometry collision mesh filename=package://mobile_manipulator_simulation/description/meshes/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; visual mesh filename=package://mobile_manipulator_simulation/description/meshes/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
- link robotiq_85_left_finger_link: geometry collision mesh filename=package://mobile_manipulator_simulation/description/meshes/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; visual mesh filename=package://mobile_manipulator_simulation/description/meshes/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
- link robotiq_85_left_finger_tip_link: geometry collision mesh filename=package://mobile_manipulator_simulation/description/meshes/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; visual mesh filename=package://mobile_manipulator_simulation/description/meshes/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
- link robotiq_85_left_inner_knuckle_link: geometry collision mesh filename=package://mobile_manipulator_simulation/description/meshes/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; visual mesh filename=package://mobile_manipulator_simulation/description/meshes/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
- link robotiq_85_left_knuckle_link: geometry collision mesh filename=package://mobile_manipulator_simulation/description/meshes/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; visual mesh filename=package://mobile_manipulator_simulation/description/meshes/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
- link robotiq_85_right_finger_link: geometry collision mesh filename=package://mobile_manipulator_simulation/description/meshes/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; visual mesh filename=package://mobile_manipulator_simulation/description/meshes/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
- link robotiq_85_right_finger_tip_link: geometry collision mesh filename=package://mobile_manipulator_simulation/description/meshes/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; visual mesh filename=package://mobile_manipulator_simulation/description/meshes/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
- link robotiq_85_right_inner_knuckle_link: geometry collision mesh filename=package://mobile_manipulator_simulation/description/meshes/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; visual mesh filename=package://mobile_manipulator_simulation/description/meshes/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
- link robotiq_85_right_knuckle_link: geometry collision mesh filename=package://mobile_manipulator_simulation/description/meshes/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; visual mesh filename=package://mobile_manipulator_simulation/description/meshes/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
- link ur5ebase_link_inertia: geometry collision mesh filename=package://mobile_manipulator_simulation/description/meshes/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; visual mesh filename=package://mobile_manipulator_simulation/description/meshes/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
- link ur5eforearm_link: geometry collision mesh filename=package://mobile_manipulator_simulation/description/meshes/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; visual mesh filename=package://mobile_manipulator_simulation/description/meshes/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
- link ur5eshoulder_link: geometry collision mesh filename=package://mobile_manipulator_simulation/description/meshes/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; visual mesh filename=package://mobile_manipulator_simulation/description/meshes/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
- link ur5eupper_arm_link: geometry collision mesh filename=package://mobile_manipulator_simulation/description/meshes/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; visual mesh filename=package://mobile_manipulator_simulation/description/meshes/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
- link ur5ewrist_1_link: geometry collision mesh filename=package://mobile_manipulator_simulation/description/meshes/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; visual mesh filename=package://mobile_manipulator_simulation/description/meshes/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
- link ur5ewrist_2_link: geometry collision mesh filename=package://mobile_manipulator_simulation/description/meshes/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; visual mesh filename=package://mobile_manipulator_simulation/description/meshes/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
- link ur5ewrist_3_link: geometry collision mesh filename=package://mobile_manipulator_simulation/description/meshes/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; visual mesh filename=package://mobile_manipulator_simulation/description/meshes/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
- link ur_to_robotiq_link: geometry collision mesh filename=package://mobile_manipulator_simulation/description/meshes/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; visual mesh filename=package://mobile_manipulator_simulation/description/meshes/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
- link wheel_left_link: geometry collision sphere radius=0.075; visual mesh filename=package://mobile_manipulator_simulation/description/meshes/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 scale=0.001 0.001 0.001
- link wheel_right_link: geometry collision sphere radius=0.075; visual mesh filename=package://mobile_manipulator_simulation/description/meshes/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 scale=0.001 0.001 0.001
Joints:
- joint wheel_left_joint: type fixed -> continuous
- joint wheel_right_joint: type fixed -> continuous
